File: hardware/light-control.kicad_pcb (KiCad board)
At the start: 2 copper layers, 50 x 35 mm, 29 parts, among them J1 PROG, J2 SWITCH, J3 INPUT, J4 OUT, Q1 BSS806, U1 LMR51610XDBVR, U2 ESP32-C3-WROOM-02-NOTHERMAL, U3 74LVC1G86

Commit message: Initial firmware version
Parts:
- R3, R4: value R -> 1k
- U1: value LMR51610XDBVR -> LMR51610YDBVR
Changed lines of the file:
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@@
     (descr "Inductor,TDK, VLS-6045, 6x6x4.5mm, https://product.tdk.com/system/files/dam/doc/product/inductor/inductor/smd/catalog/inductor_commercial_power_vls6045ex_en.pdf")
     (tags "inductor TDK VLS SMD VLS6045EF VLS6045AF")
+    (property "Part number" "VLS6045EX-220M")
     (property "Sheetfile" "light-control.kicad_sch")
     (property "Sheetname" "")
@@
         (effects (font (size 1 1) (thickness 0.15)))
     )
-    (fp_text value "R" (at 0 1.82) (layer "F.Fab")
+    (fp_text value "1k" (at 0 1.82) (layer "F.Fab")
         (effects (font (size 1 1) (thickness 0.15)))
     )
@@
         (effects (font (size 1 1) (thickness 0.15)))
     )
-    (fp_text value "LMR51610XDBVR" (at 0 2.4) (layer "F.Fab")
+    (fp_text value "LMR51610YDBVR" (at 0 2.4) (layer "F.Fab")
         (effects (font (size 1 1) (thickness 0.15)))
     )
@@
         (effects (font (size 1 1) (thickness 0.15)))
     )
-    (fp_text value "R" (at 0 1.82 90) (layer "F.Fab")
-        (effects (font (size 1 1) (thickness 0.15)))
-    )
+    (fp_text value "1k" (at 0 1.82 90) (layer "F.Fab")
+        (effects (font (size 1 1) (thickness 0.15)))
+    )
