File: hardware/light-control.kicad_sch (KiCad schematic)
At the start: 29 parts, among them J1 PROG, J2 SWITCH, J3 INPUT, J4 OUT, Q1 BSS806, U1 LMR51610XDBVR, U2 ESP32-C3-WROOM-02-NOTHERMAL, U3 74LVC1G86

Commit message: Initial firmware version
Parts:
- R3, R4: value R -> 1k
- U1: value LMR51610XDBVR -> LMR51610YDBVR; symbol lmr51606:LMR51606 -> symbols:LMR51610
- U2: symbol PCM_Espressif:ESP32-C3-WROOM-02 -> symbols:ESP32-C3-WROOM-02-NOTHERMAL
Connections:
- net GND: no longer U2.19 (GND)
